File: OneSLiPoChargerV2/OneSLiPoCharger.sch (EAGLE design)
At the start: 54 parts, among them IC1 LM358N

Commit message: Add a voltage divider on opamp output to drop voltage for the mp1584 enable pin.
Parts:
- added R3: 4.7K, rcl:R-US_0207/10
- added R4: 1K, rcl:R-US_0207/10
Connections:
- new net N$2: JP2.1, R3.1, R4.2
- net GND: now also R4.1
- net N$4: now also R3.2; no longer JP2.1
Other:
- moved on the sheet: JP2
Changed lines of the file:
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@@
 <part name="P+3" library="supply1" deviceset="+5V" device=""/>
 <part name="JP2" library="pinhead" deviceset="PINHD-1X1" device=""/>
+<part name="R3" library="rcl" deviceset="R-US_" device="0207/10" value="4.7K"/>
+<part name="R4" library="rcl" deviceset="R-US_" device="0207/10" value="1K"/>
+<part name="GND3" library="supply1" deviceset="GND" device=""/>
 </parts>
 <sheets>
@@
 <instance part="GND2" gate="1" x="68.58" y="-2.54"/>
 <instance part="P+3" gate="1" x="104.14" y="22.86"/>
-<instance part="JP2" gate="G$1" x="71.12" y="40.64"/>
+<instance part="JP2" gate="G$1" x="83.82" y="48.26"/>
+<instance part="R3" gate="G$1" x="66.04" y="40.64" rot="R180"/>
+<instance part="R4" gate="G$1" x="81.28" y="40.64" rot="R180"/>
+<instance part="GND3" gate="1" x="88.9" y="33.02"/>
 </instances>
 <busses>
@@
 <wire x1="99.06" y1="0" x2="68.58" y2="0" width="0.1524" layer="91"/>
 </segment>
+<segment>
+<pinref part="R4" gate="G$1" pin="1"/>
+<wire x1="86.36" y1="40.64" x2="88.9" y2="40.64" width="0.1524" layer="91"/>
+<wire x1="88.9" y1="40.64" x2="88.9" y2="35.56" width="0.1524" layer="91"/>
+<pinref part="GND3" gate="1" pin="GND"/>
+</segment>
 </net>
 <net name="N$4" class="0">
@@
 <wire x1="48.26" y1="55.88" x2="58.42" y2="55.88" width="0.1524" layer="91"/>
 <wire x1="58.42" y1="55.88" x2="58.42" y2="40.64" width="0.1524" layer="91"/>
-<pinref part="JP2" gate="G$1" pin="1"/>
-<wire x1="58.42" y1="40.64" x2="68.58" y2="40.64" width="0.1524" layer="91"/>
+<pinref part="R3" gate="G$1" pin="2"/>
+<wire x1="58.42" y1="40.64" x2="60.96" y2="40.64" width="0.1524" layer="91"/>
 </segment>
 </net>
@@
 </segment>
 </net>
+<net name="N$2" class="0">
+<segment>
+<pinref part="R3" gate="G$1" pin="1"/>
+<pinref part="R4" gate="G$1" pin="2"/>
+<wire x1="71.12" y1="40.64" x2="73.66" y2="40.64" width="0.1524" layer="91"/>
+<pinref part="JP2" gate="G$1" pin="1"/>
+<wire x1="73.66" y1="40.64" x2="76.2" y2="40.64" width="0.1524" layer="91"/>
+<wire x1="81.28" y1="48.26" x2="73.66" y2="48.26" width="0.1524" layer="91"/>
+<wire x1="73.66" y1="48.26" x2="73.66" y2="40.64" width="0.1524" layer="91"/>
+</segment>
+</net>
