File: ReflowCntrl/ReflowCntrl.sch (EAGLE design)
At the start: 13 parts, among them J1 DCJ0202, T1 2N2222, X1 1751248

Commit message: Fix swapped VCC and GND pins on OLED. Resized board a bit.
Connections:
- net GND: now also JP1.1; no longer JP1.2
- net VCC: now also JP1.2; no longer JP1.1
Changed lines of the file:
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@@
-</segment>
-<segment>
-<pinref part="JP1" gate="A" pin="2"/>
-<wire x1="104.14" y1="86.36" x2="93.98" y2="86.36" width="0.1524" layer="91"/>
-<label x="93.98" y="86.36" size="1.778" layer="95" rot="R180" xref="yes"/>
 </segment>
 <segment>
@@
 <pinref part="GND7" gate="1" pin="GND"/>
 </segment>
+<segment>
+<pinref part="JP1" gate="A" pin="1"/>
+<wire x1="104.14" y1="88.9" x2="93.98" y2="88.9" width="0.1524" layer="91"/>
+<label x="93.98" y="88.9" size="1.778" layer="95" rot="R180" xref="yes"/>
+</segment>
 </net>
 <net name="VCC" class="0">
@@
 <pinref part="SG1" gate="G$1" pin="1"/>
 <wire x1="25.4" y1="22.86" x2="25.4" y2="17.78" width="0.1524" layer="91"/>
-</segment>
-<segment>
-<pinref part="JP1" gate="A" pin="1"/>
-<wire x1="104.14" y1="88.9" x2="93.98" y2="88.9" width="0.1524" layer="91"/>
-<label x="93.98" y="88.9" size="1.778" layer="95" rot="R180" xref="yes"/>
 </segment>
 <segment>
@@
 <pinref part="P+5" gate="VCC" pin="VCC"/>
 </segment>
+<segment>
+<pinref part="JP1" gate="A" pin="2"/>
+<wire x1="104.14" y1="86.36" x2="93.98" y2="86.36" width="0.1524" layer="91"/>
+<label x="93.98" y="86.36" size="1.778" layer="95" rot="R180" xref="yes"/>
+</segment>
 </net>

Commit message: Change SSR terminal to Wago part.
Parts:
- removed X1: 1751248, con-phoenix-350:1751248
- added X2: (no value), con-wago-508:W237-02P
Connections:
- net GND: now also X2-1.KL; no longer X1-1.K
- net SSR: now also X2-2.KL; no longer X1-2.K
Changed lines of the file:
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@@
 <part name="T1" library="adafruit" deviceset="2N2222" device=""/>
 <part name="SG1" library="buzzer" deviceset="F/CM12P" device=""/>
-<part name="X1" library="con-phoenix-350" deviceset="1751248" device=""/>
 <part name="U$1" library="LM7805" deviceset="7805-TO220V" device=""/>
 <part name="J1" library="con-jack-jke" deviceset="DCJ0202" device=""/>
@@
 <part name="GND6" library="supply1" deviceset="GND" device=""/>
 <part name="GND7" library="supply1" deviceset="GND" device=""/>
+<part name="X2" library="con-wago-508" deviceset="W237-02P" device=""/>
 </parts>
 <sheets>
@@
 <instance part="T1" gate="G$1" x="22.86" y="-2.54"/>
 <instance part="SG1" gate="G$1" x="27.94" y="15.24" rot="R270"/>
-<instance part="X1" gate="-1" x="124.46" y="50.8" rot="R180"/>
-<instance part="X1" gate="-2" x="124.46" y="55.88" rot="R180"/>
 <instance part="U$1" gate="G$1" x="7.62" y="78.74"/>
 <instance part="J1" gate="G$1" x="-10.16" y="78.74"/>
@@
 <instance part="GND6" gate="1" x="30.48" y="66.04"/>
 <instance part="GND7" gate="1" x="45.72" y="22.86"/>
+<instance part="X2" gate="-1" x="121.92" y="50.8"/>
+<instance part="X2" gate="-2" x="121.92" y="55.88"/>
 </instances>
 <busses>
@@
 </segment>
 <segment>
-<pinref part="X1" gate="-1" pin="K"/>
 <pinref part="GND5" gate="1" pin="GND"/>
 <wire x1="127" y1="50.8" x2="134.62" y2="50.8" width="0.1524" layer="91"/>
+<pinref part="X2" gate="-1" pin="KL"/>
 </segment>
 <segment>
@@
 </segment>
 <segment>
-<pinref part="X1" gate="-2" pin="K"/>
 <wire x1="127" y1="55.88" x2="132.08" y2="55.88" width="0.1524" layer="91"/>
 <label x="132.08" y="55.88" size="1.778" layer="95" xref="yes"/>
-</segment>
-</net>
+<pinref part="X2" gate="-2" pin="KL"/>
+</segment>
+</net>

Commit message: Change resistors to 0207/10 package
Parts:
- R1, R2, R3: device rcl:R-US_0204/5 -> rcl:R-US_0207/10
Changed lines of the file:
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@@
 <part name="S1" library="switch-omron" deviceset="10-XX" device=""/>
 <part name="S2" library="switch-omron" deviceset="10-XX" device=""/>
-<part name="R1" library="rcl" deviceset="R-US_" device="0204/5"/>
-<part name="R2" library="rcl" deviceset="R-US_" device="0204/5"/>
+<part name="R1" library="rcl" deviceset="R-US_" device="0207/10"/>
+<part name="R2" library="rcl" deviceset="R-US_" device="0207/10"/>
 <part name="JP1" library="pinhead" deviceset="PINHD-1X4" device="" value="OLED"/>
 <part name="JP2" library="pinhead" deviceset="PINHD-1X5" device="" value="Thermo"/>
@@
 <part name="U$1" library="LM7805" deviceset="7805-TO220V" device=""/>
 <part name="J1" library="con-jack-jke" deviceset="DCJ0202" device=""/>
-<part name="R3" library="rcl" deviceset="R-US_" device="0204/5"/>
+<part name="R3" library="rcl" deviceset="R-US_" device="0207/10"/>
 <part name="GND1" library="supply1" deviceset="GND" device=""/>
 <part name="P+1" library="supply1" deviceset="VCC" device=""/>
