File: PicTouchTest/PicTouchTest.sch (EAGLE design)
At the start: 9 parts

Commit message: Increase the touch button size to 20mm diameter.
Parts:
- U$2, U$3, U$4, U$5, U$6, U$7: value CAPTOUCH -> CAPTOUCH20MMRND; device CapTouch:CAPTOUCH -> CapTouch:CAPTOUCH20MMRND
Changed lines of the file:
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@@
 <part name="P+1" library="supply1" deviceset="VCC" device=""/>
 <part name="PK3HDR" library="pinhead" deviceset="PINHD-1X6" device=""/>
-<part name="U$2" library="CapTouch" deviceset="CAPTOUCH" device=""/>
-<part name="U$3" library="CapTouch" deviceset="CAPTOUCH" device=""/>
-<part name="U$4" library="CapTouch" deviceset="CAPTOUCH" device=""/>
-<part name="U$5" library="CapTouch" deviceset="CAPTOUCH" device=""/>
-<part name="U$6" library="CapTouch" deviceset="CAPTOUCH" device=""/>
-<part name="U$7" library="CapTouch" deviceset="CAPTOUCH" device=""/>
+<part name="U$2" library="CapTouch" deviceset="CAPTOUCH" device="20MMRND" value="CAPTOUCH20MMRND"/>
+<part name="U$3" library="CapTouch" deviceset="CAPTOUCH" device="20MMRND" value="CAPTOUCH20MMRND"/>
+<part name="U$4" library="CapTouch" deviceset="CAPTOUCH" device="20MMRND" value="CAPTOUCH20MMRND"/>
+<part name="U$5" library="CapTouch" deviceset="CAPTOUCH" device="20MMRND" value="CAPTOUCH20MMRND"/>
+<part name="U$6" library="CapTouch" deviceset="CAPTOUCH" device="20MMRND" value="CAPTOUCH20MMRND"/>
+<part name="U$7" library="CapTouch" deviceset="CAPTOUCH" device="20MMRND" value="CAPTOUCH20MMRND"/>
 <part name="I2CHDR" library="pinhead" deviceset="PINHD-1X4" device=""/>
 <part name="P+2" library="supply1" deviceset="VCC" device=""/>
