File: NixieClockDisplay/NixieClockDisplay.brd (EAGLE design)
At the start: 121.9 x 69.8 mm, 15 parts

Commit message: Bunch of random updated
Other:
- board text added: "Huskymutt Nixie Display v0.2 Sept 17, 2017"
Changed lines of the file:
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@@
 <layer number="23" name="tOrigins" color="15" fill="1" visible="yes" active="yes"/>
 <layer number="24" name="bOrigins" color="15" fill="1" visible="yes" active="yes"/>
-<layer number="25" name="tNames" color="7" fill="1" visible="no" active="yes"/>
-<layer number="26" name="bNames" color="7" fill="1" visible="no" active="yes"/>
+<layer number="25" name="tNames" color="7" fill="1" visible="yes" active="yes"/>
+<layer number="26" name="bNames" color="7" fill="1" visible="yes" active="yes"/>
 <layer number="27" name="tValues" color="7" fill="1" visible="no" active="yes"/>
 <layer number="28" name="bValues" color="7" fill="1" visible="no" active="yes"/>
@@
 <hole x="4.445" y="34.925" drill="3.2766"/>
 <hole x="117.475" y="34.925" drill="3.2766"/>
+<text x="59.055" y="31.75" size="1.778" layer="22" rot="MR90">Huskymutt Nixie Display v0.2
+Sept 17, 2017</text>
 </plain>
 <attributes>
@@
 </board>
 </drawing>
+<compatibility>
+<note version="6.3" minversion="6.2.2" severity="warning">
+Since Version 6.2.2 text objects can contain more than one line,
+which will not be processed correctly with this version.
+</note>
+</compatibility>
 </eagle>
