File: NixieClockControllerWemos/NixieClockControllerWemos.brd (EAGLE design)
At the start: 121.9 x 38.1 mm, 25 parts, among them IC1 NE555, Q1 BUZ11BV, T1 BC547

Commit message: Fix LM317 wiring and add hex inverter.
Parts:
- added IC2: 74HCT04N, 74xx-eu:DIL14
- moved X1 35.3 mm to (72.4, 33.0), turned to 0 degrees
- moved R7 25.6 mm to (54.6, 7.62), turned to 270 degrees
- moved Q1 24.1 mm to (85.1, 35.6), turned to 0 degrees
- moved R9 18.0 mm to (55.9, 30.5)
- moved R10 13.7 mm to (52.1, 30.5)
- moved U$3 13.5 mm to (64.8, 27.9)
- moved CONF 11.7 mm to (54.6, 17.8)
- moved WEMOS1 7.62 mm to (33.0, 20.3)
Connections:
- new net N$17: IC2.13, WEMOS1.D0
- new net N$18: IC2.11, WEMOS1.D5
- new net N$19: IC2.3, WEMOS1.D6
- new net N$20: IC2.5, WEMOS1.D7
- new net N$21: IC2.9, WEMOS1.D8
- net 5V: now also IC2.14, R9.1; no longer R9.2
- net GND: now also IC2.7, R10.2; no longer R10.1, U$3.ADJ
- net N$11: now also IC2.10; no longer WEMOS1.D5
- net N$12: now also R10.1, R9.2, U$3.ADJ; no longer R10.2, R9.1
- net N$13: now also IC2.4; no longer WEMOS1.D6
- net N$14: now also IC2.6; no longer WEMOS1.D7
- net N$15: now also IC2.8; no longer WEMOS1.D8
- net N$5: now also IC2.12; no longer WEMOS1.D0
Routing:
- net N$1: track 15.0 -> 33.9 mm
- net N$2: track 50.2 -> 32.4 mm
- net N$19: track 0.00 -> 14.8 mm
- net N$20: track 0.00 -> 13.8 mm
- net N$12: track 3.81 -> 13.8 mm
- net 5V: track 99.3 -> 108.9 mm
- net N$18: track 0.00 -> 6.13 mm
- net VCC: track 122.3 -> 128.1 mm
- net N$11: track 11.2 -> 16.6 mm
- net N$13: track 11.2 -> 6.13 mm
- net N$21: track 0.00 -> 5.08 mm
- net N$17: track 0.00 -> 5.08 mm
- net N$15: track 11.2 -> 15.5 mm
- net N$14: track 11.2 -> 7.18 mm
- net N$5: track 11.2 -> 14.8 mm
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
Commit message: Add a voltage regulator.
Other:
- board text added: "Huskymutt Nixie Control Wemos v0.2 Oct 22, 2017"
- board text removed: "Huskymutt Nixie Control Wemos v0.1 Sept 17, 2017"
Changed lines of the file:
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@@
 <layer number="23" name="tOrigins" color="15" fill="1" visible="yes" active="yes"/>
 <layer number="24" name="bOrigins" color="15" fill="1" visible="yes" active="yes"/>
-<layer number="25" name="tNames" color="7" fill="1" visible="yes" active="yes"/>
-<layer number="26" name="bNames" color="7" fill="1" visible="yes" active="yes"/>
-<layer number="27" name="tValues" color="7" fill="1" visible="yes" active="yes"/>
-<layer number="28" name="bValues" color="7" fill="1" visible="yes" active="yes"/>
+<layer number="25" name="tNames" color="7" fill="1" visible="no" active="yes"/>
+<layer number="26" name="bNames" color="7" fill="1" visible="no" active="yes"/>
+<layer number="27" name="tValues" color="7" fill="1" visible="no" active="yes"/>
+<layer number="28" name="bValues" color="7" fill="1" visible="no" active="yes"/>
 <layer number="29" name="tStop" color="7" fill="3" visible="no" active="yes"/>
 <layer number="30" name="bStop" color="7" fill="6" visible="no" active="yes"/>
@@
 <layer number="37" name="tTest" color="7" fill="1" visible="no" active="yes"/>
 <layer number="38" name="bTest" color="7" fill="1" visible="no" active="yes"/>
-<layer number="39" name="tKeepout" color="4" fill="11" visible="yes" active="yes"/>
-<layer number="40" name="bKeepout" color="1" fill="11" visible="yes" active="yes"/>
-<layer number="41" name="tRestrict" color="4" fill="10" visible="yes" active="yes"/>
-<layer number="42" name="bRestrict" color="1" fill="10" visible="yes" active="yes"/>
-<layer number="43" name="vRestrict" color="2" fill="10" visible="yes" active="yes"/>
+<layer number="39" name="tKeepout" color="4" fill="11" visible="no" active="yes"/>
+<layer number="40" name="bKeepout" color="1" fill="11" visible="no" active="yes"/>
+<layer number="41" name="tRestrict" color="4" fill="10" visible="no" active="yes"/>
+<layer number="42" name="bRestrict" color="1" fill="10" visible="no" active="yes"/>
+<layer number="43" name="vRestrict" color="2" fill="10" visible="no" active="yes"/>
 <layer number="44" name="Drills" color="7" fill="1" visible="no" active="yes"/>
-<layer number="45" name="Holes" color="7" fill="1" visible="yes" active="yes"/>
+<layer number="45" name="Holes" color="7" fill="1" visible="no" active="yes"/>
 <layer number="46" name="Milling" color="3" fill="1" visible="no" active="yes"/>
 <layer number="47" name="Measures" color="7" fill="1" visible="no" active="yes"/>
-<layer number="48" name="Document" color="7" fill="1" visible="yes" active="yes"/>
-<layer number="49" name="Reference" color="7" fill="1" visible="yes" active="yes"/>
-<layer number="51" name="tDocu" color="7" fill="1" visible="yes" active="yes"/>
-<layer number="52" name="bDocu" color="7" fill="1" visible="yes" active="yes"/>
+<layer number="48" name="Document" color="7" fill="1" visible="no" active="yes"/>
+<layer number="49" name="Reference" color="7" fill="1" visible="no" active="yes"/>
+<layer number="51" name="tDocu" color="7" fill="1" visible="no" active="yes"/>
+<layer number="52" name="bDocu" color="7" fill="1" visible="no" active="yes"/>
 <layer number="90" name="Modules" color="5" fill="1" visible="no" active="no"/>
 <layer number="91" name="Nets" color="2" fill="1" visible="no" active="no"/>
@@
 <hole x="4.445" y="4.445" drill="3.2766"/>
 <hole x="117.475" y="4.445" drill="3.2766"/>
-<text x="110.49" y="31.75" size="1.778" layer="22" rot="MR0">Huskymutt Nixie Control Wemos v0.1
-Sept 17, 2017</text>
+<text x="110.49" y="31.75" size="1.778" layer="22" rot="MR0">Huskymutt Nixie Control Wemos v0.2
+Oct 22, 2017</text>
 </plain>
 <attributes>
