File: OneSLiPoChargerV3/OneSLiPoCharger.brd (EAGLE design)
At the start: 86.4 x 52.1 mm, 62 parts, among them IC1 LM358N

Commit message: Bunch of random updated
Other:
- board text added: "Huskymutt 1S charger V3.0 Sept 17, 2017"
Changed lines of the file:
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@@
 <wire x1="22.352" y1="23.368" x2="22.352" y2="24.384" width="0.1016" layer="146"/>
 <text x="45.72" y="22.86" size="1.016" layer="21">BAT4</text>
+<text x="74.93" y="24.13" size="1.778" layer="22" rot="MR0">Huskymutt 1S charger V3.0
+Sept 17, 2017</text>
 </plain>
 <attributes>
@@
 </drawing>
 <compatibility>
+<note version="6.3" minversion="6.2.2" severity="warning">
+Since Version 6.2.2 text objects can contain more than one line,
+which will not be processed correctly with this version.
+</note>
 <note version="8.2" severity="warning">
 Since Version 8.2, Eagle supports online libraries. The ids
